Commit message: added meshes and only use stl in urdf

File: urdf/starter_kit.urdf.xacro (robot description, xacro)
@@ -5,5 +5,5 @@
       <visual>
         <geometry>
-          <mesh filename="package://cpr_onav_description/meshes/starter_kit.dae" />
+          <mesh filename="package://cpr_onav_description/meshes/starter_kit.stl" />
         </geometry>
       </visual>

Commit message: remove commented color

File: urdf/starter_kit.urdf.xacro (robot description, xacro)
@@ -9,8 +9,4 @@
         </geometry>
         <material name="yellow" />
-<!--         <material name="yellow" >
-          <color rgba="255 237 4 1" />
-        </material>
--->
         <origin xyz="0 0 0" rpy="0 0 0" />
       </visual>
