Commit message: Fix the paths to the wibotic antenna mesh

File: urdf/husky_observer.urdf.xacro (robot description, xacro)
@@ -76,5 +76,5 @@
     <visual>
       <geometry>
-        <mesh filename="package://husky_observer_description/meshes/wibotic.stl" />
+        <mesh filename="package://cpr_onav_description/meshes/wibotic.stl" />
       </geometry>
       <material name="black" />
@@ -83,5 +83,5 @@
     <collision>
       <geometry>
-        <mesh filename="package://husky_observer_description/meshes/wibotic.stl" />
+        <mesh filename="package://cpr_onav_description/meshes/wibotic.stl" />
       </geometry>
       <origin xyz="0 0 0" rpy="0 0 0" />

Commit message: Add coloured cylinders to represent the two sections of the stack light

File: urdf/husky_observer.urdf.xacro (robot description, xacro)
@@ -56,4 +56,22 @@
       <origin xyz="-0.28 0 0.7675" />
     </collision>
+    <visual>
+      <geometry>
+        <cylinder radius="0.036" length="0.045" />
+      </geometry>
+      <material name="orange_glow">
+        <color rgba="1 0.8 0 1" />
+      </material>
+      <origin xyz="-0.27 0 0.75" rpy="0 0 0" />
+    </visual>
+    <visual>
+      <geometry>
+        <cylinder radius="0.036" length="0.064" />
+      </geometry>
+      <material name="white_glow">
+        <color rgba="1 1 1 1" />
+      </material>
+      <origin xyz="-0.27 0 0.827" rpy="0 0 0" />
+    </visual>
     <collision>
       <!-- camera mount -->
