Commit message: added velodyne dae file. fix swiftnav heading xyz var

File: urdf/outdoornav_description.urdf.xacro (robot description, xacro)
@@ -1,5 +1,4 @@
 <?xml version="1.0"?>
 <robot xmlns:xacro="http://ros.org/wiki/xacro" name="outdoornav_sensors">
-  <!-- <xacro:macro name="outdoornav_sensors" params="starter_kit_configuration standard_kit_configuration custom_configuration"> -->
   <xacro:macro name="outdoornav_sensors" params="outdoornav_configuration">
     <xacro:arg name="starter_kit_xyz"          default="$(optenv STARTER_KIT_XYZ 0.0 0.0 0.0)" />
@@ -55,5 +54,4 @@
     <xacro:arg name="onav_urdf_extras"         default="$(optenv OUTDOORNAV_URDF_EXTRAS empty.urdf)" />
     <!-- Starter Kit -->
-    <!-- <xacro:if value="${starter_kit_configuration}"> -->
     <xacro:if value="${outdoornav_configuration == 'starter'}">
       <xacro:include filename="$(find cpr_onav_description)/urdf/starter_kit.urdf.xacro" />
@@ -74,10 +72,9 @@
     </xacro:if>
     <!-- Standard Kit -->
-    <!-- <xacro:if value="${standard_kit_configuration}"> -->
     <xacro:if value="${outdoornav_configuration == 'standard'}">
       <xacro:include filename="$(find cpr_onav_description)/urdf/standard_kit.urdf.xacro" />
       <xacro:standard_kit
         swiftnav_position_xyz="$(arg swiftnav_position_xyz)"
-        swiftnav_heading_rpy="$(arg swiftnav_heading_rpy)"
+        swiftnav_heading_xyz="$(arg swiftnav_heading_xyz)"
         microstrain_xyz="$(arg microstrain_xyz)"
         microstrain_rpy="$(arg microstrain_rpy)"
@@ -87,5 +84,4 @@
     </xacro:if>
     <!-- Custom configuration -->
-    <!-- <xacro:if value="${custom_configuration}"> -->
     <xacro:if value="${outdoornav_configuration == 'custom'}">
       <!-- Position GPS (Duro) -->
@@ -136,5 +132,16 @@
       <!-- Velodyne Link -->
       <xacro:if value="$(arg vlp_enable)">
-        <link name="velodyne"/>
+        <link name="velodyne">
+          <visual>
+            <geometry>
+              <mesh filename="package://velodyne_description/meshes/VLP16_scan.dae" />
+            </geometry>
+          </visual>
+          <visual>
+            <geometry>
+              <mesh filename="package://velodyne_description/meshes/VLP16_scan.dae" />
+            </geometry>
+          </visual>
+        </link>
         <joint name="velodyne_to_base" type="fixed">
           <parent link="base_link" />
@@ -145,5 +152,16 @@
       <!-- Rear Velodyne Link -->
       <xacro:if value="$(arg rear_vlp_enable)">
-        <link name="rear_velodyne"/>
+        <link name="rear_velodyne">
+          <visual>
+            <geometry>
+              <mesh filename="package://velodyne_description/meshes/VLP16_scan.dae" />
+            </geometry>
+          </visual>
+          <visual>
+            <geometry>
+              <mesh filename="package://velodyne_description/meshes/VLP16_scan.dae" />
+            </geometry>
+          </visual>
+        </link>
         <joint name="rear_velodyne_to_base" type="fixed">
           <parent link="base_link" />
@@ -220,5 +238,5 @@
         </joint>
       </xacro:if>
-      <!-- Optinal for OEM platforms or additional sensors customers want to use as inputs to OutdoorNav -->
+      <!-- Optional for OEM platforms or additional sensors customers want to use as inputs to OutdoorNav -->
       <xacro:include filename="$(arg onav_urdf_extras)" />
     </xacro:if>

File: urdf/standard_kit.urdf.xacro (robot description, xacro)
@@ -24,5 +24,16 @@
     </joint>
     <!-- Velodyne Link -->
-    <link name="velodyne"/>
+    <link name="velodyne">
+      <visual>
+        <geometry>
+          <mesh filename="package://velodyne_description/meshes/VLP16_scan.dae" />
+        </geometry>
+      </visual>
+      <visual>
+        <geometry>
+          <mesh filename="package://velodyne_description/meshes/VLP16_scan.dae" />
+        </geometry>
+      </visual>
+    </link>
     <joint name="velodyne_to_base" type="fixed">
       <parent link="base_link" />

Commit message: tested urdf initialization with all config types

File: urdf/outdoornav_description.urdf.xacro (robot description, xacro)
@@ -25,13 +25,17 @@
     <xacro:arg name="lms1xx_xyz"               default="$(optenv LMS1XX_XYZ 0.0 0.0 0.0)" />
     <xacro:arg name="lms1xx_rpy"               default="$(optenv LMS1XX_RPY 0.0 0.0 0.0)" />
+    <xacro:arg name="lms1xx_num"               default="$(optenv LMS1XX_NUM 0)" />
     <xacro:arg name="rear_lms1xx_enable"       default="$(optenv REAR_LMS1XX_ENABLE_DRIVER false)" />
     <xacro:arg name="rear_lms1xx_xyz"          default="$(optenv REAR_LMS1XX_XYZ 0.0 0.0 0.0)" />
     <xacro:arg name="rear_lms1xx_rpy"          default="$(optenv REAR_LMS1XX_RPY 0.0 0.0 0.0)" />
+    <xacro:arg name="rear_lms1xx_num"          default="$(optenv REAR_LMS1XX_NUM 0)" />
     <xacro:arg name="hokuyo_enable"            default="$(optenv HOKUYO_ENABLE_DRIVER false)" />
     <xacro:arg name="hokuyo_xyz"               default="$(optenv HOKUYO_XYZ 0.0 0.0 0.0)" />
     <xacro:arg name="hokuyo_rpy"               default="$(optenv HOKUYO_RPY 0.0 0.0 0.0)" />
+    <xacro:arg name="hokuyo_num"               default="$(optenv HOKUYO_NUM 0)" />
     <xacro:arg name="rear_hokuyo_enable"       default="$(optenv REAR_HOKUYO_ENABLE_DRIVER false)" />
     <xacro:arg name="rear_hokuyo_xyz"          default="$(optenv REAR_HOKUYO_XYZ 0.0 0.0 0.0)" />
     <xacro:arg name="rear_hokuyo_rpy"          default="$(optenv REAR_HOKUYO_RPY 0.0 0.0 0.0)" />
+    <xacro:arg name="rear_hokuyo_num"          default="$(optenv REAR_HOKUYO_NUM 0)" />
     <xacro:arg name="outdoorscan_enable"       default="$(optenv OUTDOORSCAN_ENABLE_DRIVER false)" />
     <xacro:arg name="outdoorscan_xyz"          default="$(optenv OUTDOORSCAN_XYZ 0.0 0.0 0.0)" />
@@ -43,4 +47,5 @@
     <xacro:arg name="vlp_xyz"                  default="$(optenv VLP_XYZ 0.0 0.0 0.0)" />
     <xacro:arg name="vlp_rpy"                  default="$(optenv VLP_RPY 0.0 0.0 0.0)" />
+    <xacro:arg name="vlp_num"                  default="$(optenv VLP_NUM 0)" />
     <xacro:arg name="rear_vlp_enable"          default="$(optenv REAR_VLP_ENABLE_DRIVER false)" />
     <xacro:arg name="rear_vlp_xyz"             default="$(optenv REAR_VLP_XYZ 0.0 0.0 0.0)" />
@@ -80,9 +85,14 @@
         microstrain_rpy="$(arg microstrain_rpy)"
         vlp_xyz="$(arg vlp_xyz)"
-        vlp_rpy="$(arg vlp_rpy)" >
+        vlp_rpy="$(arg vlp_rpy)"
+        vlp_num="$(arg vlp_num)" >
       </xacro:standard_kit>
     </xacro:if>
     <!-- Custom configuration -->
     <xacro:if value="${outdoornav_configuration == 'custom'}">
+      <xacro:include filename="$(find velodyne_description)/urdf/VLP-16.urdf.xacro"/>
+      <xacro:include filename="$(find husky_description)/urdf/accessories/hokuyo_ust10.urdf.xacro" />
+      <xacro:include filename="$(find husky_description)/urdf/accessories/sick_lms1xx_mount.urdf.xacro"/>
+      <xacro:include filename="$(find realsense2_description)/urdf/_d435.urdf.xacro" />
       <!-- Position GPS (Duro) -->
       <xacro:if value="$(arg swiftnav_position_enable)">
@@ -132,59 +142,24 @@
       <!-- Velodyne Link -->
       <xacro:if value="$(arg vlp_enable)">
-        <link name="velodyne">
-          <visual>
-            <geometry>
-              <mesh filename="package://velodyne_description/meshes/VLP16_scan.dae" />
-            </geometry>
-          </visual>
-          <visual>
-            <geometry>
-              <mesh filename="package://velodyne_description/meshes/VLP16_scan.dae" />
-            </geometry>
-          </visual>
-        </link>
-        <joint name="velodyne_to_base" type="fixed">
-          <parent link="base_link" />
-          <child link="velodyne" />
-          <origin xyz="$(arg vlp_xyz)" rpy="$(arg vlp_rpy)"/>
-        </joint>
+        <xacro:VLP-16 name="velodyne" parent="base_link" topic="/sensors/lidar/$(arg vlp_num)/pointcloud">
+          <origin xyz="$(arg vlp_xyz)" rpy="$(arg vlp_rpy)" />
+        </xacro:VLP-16>
       </xacro:if>
       <!-- Rear Velodyne Link -->
       <xacro:if value="$(arg rear_vlp_enable)">
-        <link name="rear_velodyne">
-          <visual>
-            <geometry>
-              <mesh filename="package://velodyne_description/meshes/VLP16_scan.dae" />
-            </geometry>
-          </visual>
-          <visual>
-            <geometry>
-              <mesh filename="package://velodyne_description/meshes/VLP16_scan.dae" />
-            </geometry>
-          </visual>
-        </link>
-        <joint name="rear_velodyne_to_base" type="fixed">
-          <parent link="base_link" />
-          <child link="rear_velodyne" />
-          <origin xyz="$(arg rear_vlp_xyz)" rpy="$(arg rear_vlp_rpy)"/>
-        </joint>
+        <xacro:VLP-16 name="rear_velodyne" parent="base_link" topic="/sensors/lidar/$(arg vlp_num)/pointcloud">
+          <origin xyz="$(arg rear_vlp_xyz)" rpy="$(arg rear_vlp_rpy)" />
+        </xacro:VLP-16>
       </xacro:if>
       <!-- 2D LiDAR(s) Link -->
       <xacro:if value="$(arg lms1xx_enable)">
-        <xacro:include filename="$(find husky_description)/urdf/accessories/sick_lms1xx_mount.urdf.xacro"/>
-        <link name="front_laser"/>
-        <joint name="front_laser_to_base" type="fixed">
-          <parent link="base_link" />
-          <child link="front_laser" />
+        <xacro:sick_lms1xx_mount prefix="front" parent="base_link" topic="/sensors/lidar/$(arg lms1xx_num)/scan" tower="0" robot_namespace="/">
           <origin xyz="$(arg lms1xx_xyz)" rpy="$(arg lms1xx_rpy)"/>
-        </joint>
+        </xacro:sick_lms1xx_mount>
       </xacro:if>
       <xacro:if value="$(arg hokuyo_enable)">
-        <link name="front_laser"/>
-        <joint name="front_laser_to_base" type="fixed">
-          <parent link="base_link" />
-          <child link="front_laser" />
-          <origin xyz="$(arg hokuyo_xyz)" rpy="$(arg hokuyo_rpy)"/>
-        </joint>
+        <xacro:hokuyo_ust10_mount prefix="front_laser" parent_link="base_link" topic="/sensors/lidar/$(arg hokuyo_num)/scan">
+            <origin xyz="$(arg hokuyo_xyz)" rpy="$(arg hokuyo_rpy)" />
+        </xacro:hokuyo_ust10_mount>
       </xacro:if>
       <xacro:if value="$(arg outdoorscan_enable)">
@@ -198,18 +173,12 @@
       <!-- Rear 2D LiDAR(s) Link -->
       <xacro:if value="$(arg rear_lms1xx_enable)">
-        <link name="rear_laser"/>
-        <joint name="rear_laser_to_base" type="fixed">
-          <parent link="base_link" />
-          <child link="rear_laser" />
-          <origin xyz="$(arg rear_lms1xx_xyz)" rpy="$(arg rear_lms1xx_rpy)"/>
-        </joint>
+        <xacro:sick_lms1xx_mount prefix="rear" parent="base_link" topic="/sensors/lidar/$(arg rear_lms1xx_num)/scan" tower="0" robot_namespace="/">
+          <origin xyz="$(arg lms1xx_xyz)" rpy="$(arg lms1xx_rpy)"/>
+        </xacro:sick_lms1xx_mount>
       </xacro:if>
       <xacro:if value="$(arg rear_hokuyo_enable)">
-        <link name="rear_laser"/>
-        <joint name="rear_laser_to_base" type="fixed">
-          <parent link="base_link" />
-          <child link="rear_laser" />
-          <origin xyz="$(arg rear_hokuyo_xyz)" rpy="$(arg rear_hokuyo_rpy)"/>
-        </joint>
+        <xacro:hokuyo_ust10_mount prefix="rear_laser" parent_link="base_link" topic="/sensors/lidar/$(arg rear_hokuyo_num)/scan">
+            <origin xyz="$(arg hokuyo_xyz)" rpy="$(arg hokuyo_rpy)" />
+        </xacro:hokuyo_ust10_mount>
       </xacro:if>
       <xacro:if value="$(arg rear_outdoorscan_enable)">
@@ -223,18 +192,12 @@
       <!-- Realsense D435 Link -->
       <xacro:if value="$(arg d435_enable)">
-        <link name="front_d435_link"/>
-        <joint name="front_d435_to_base" type="fixed">
-          <parent link="base_link" />
-          <child link="front_d435_link" />
+        <xacro:sensor_d435 name="front_d435" parent="base_link" use_mesh="true">
           <origin xyz="$(arg d435_xyz)" rpy="$(arg d435_rpy)"/>
-        </joint>
+        </xacro:sensor_d435>
       </xacro:if>
       <xacro:if value="$(arg rear_d435_enable)">
-        <link name="rear_d435_link"/>
-        <joint name="rear_d435_to_base" type="fixed">
-          <parent link="base_link" />
-          <child link="rear_d435_link" />
+        <xacro:sensor_d435 name="rear_d435" parent="base_link" use_mesh="true">
           <origin xyz="$(arg rear_d435_xyz)" rpy="$(arg rear_d435_rpy)"/>
-        </joint>
+        </xacro:sensor_d435>
       </xacro:if>
       <!-- Optional for OEM platforms or additional sensors customers want to use as inputs to OutdoorNav -->

File: urdf/standard_kit.urdf.xacro (robot description, xacro)
@@ -1,18 +1,51 @@
 <?xml version="1.0"?>
 <robot xmlns:xacro="http://ros.org/wiki/xacro" name="cpr_onav_standard_kit">
-  <xacro:macro name="standard_kit" params="swiftnav_position_xyz swiftnav_heading_xyz microstrain_xyz microstrain_rpy vlp_xyz vlp_rpy">
+  <xacro:macro name="standard_kit" params="swiftnav_position_xyz swiftnav_heading_xyz microstrain_xyz microstrain_rpy vlp_xyz vlp_rpy vlp_num">
+    <xacro:include filename="$(find velodyne_description)/urdf/VLP-16.urdf.xacro"/>
     <!-- Position GPS (Duro) -->
-    <link name="gps_position_link"/>
+    <link name="gps_position_link">
+      <visual>
+        <geometry>
+          <mesh filename="package://cpr_onav_description/meshes/gnss_antenna.stl" />
+        </geometry>
+        <origin xyz="0 0 0" rpy="0 0 0" />
+        <material name="white">
+          <color rgba="1 1 1 1" />
+        </material>
+      </visual>
+      <collision>
+        <geometry>
+          <mesh filename="package://cpr_onav_description/meshes/gnss_antenna.stl" />
+        </geometry>
+        <origin xyz="0 0 0" rpy="0 0 0 " />
+      </collision>
+    </link>
     <joint name="gps_position_to_base" type="fixed">
       <parent link="base_link" />
       <child link="gps_position_link" />
-      <origin xyz="$(arg swiftnav_position_xyz)" rpy="0.0 0.0 0.0"/>
+      <origin xyz="${swiftnav_position_xyz}" rpy="0 0 0"/>
     </joint>
     <!-- Heading GPS -->
-    <link name="gps_heading_link"/>
+    <link name="gps_heading_link">
+      <visual>
+        <geometry>
+          <mesh filename="package://cpr_onav_description/meshes/gnss_antenna.stl" />
+        </geometry>
+        <origin xyz="0 0 0" rpy="0 0 0" />
+        <material name="white">
+          <color rgba="1 1 1 1" />
+        </material>
+      </visual>
+      <collision>
+        <geometry>
+          <mesh filename="package://cpr_onav_description/meshes/gnss_antenna.stl" />
+        </geometry>
+        <origin xyz="0 0 0" rpy="0 0 0 " />
+      </collision>
+    </link>
     <joint name="gps_heading_to_base" type="fixed">
       <parent link="base_link" />
       <child link="gps_heading_link" />
-      <origin xyz="$(arg swiftnav_heading_xyz)" rpy="0.0 0.0 0.0"/>
+      <origin xyz="${swiftnav_heading_xyz}" rpy="0 0 0"/>
     </joint>
     <!-- Microstrain Link -->
@@ -21,24 +54,10 @@
       <parent link="base_link" />
       <child link="microstrain_link" />
-      <origin xyz="$(arg microstrain_xyz)" rpy="$(arg microstrain_rpy)"/>
+      <origin xyz="${microstrain_xyz}" rpy="${microstrain_rpy}"/>
     </joint>
     <!-- Velodyne Link -->
-    <link name="velodyne">
-      <visual>
-        <geometry>
-          <mesh filename="package://velodyne_description/meshes/VLP16_scan.dae" />
-        </geometry>
-      </visual>
-      <visual>
-        <geometry>
-          <mesh filename="package://velodyne_description/meshes/VLP16_scan.dae" />
-        </geometry>
-      </visual>
-    </link>
-    <joint name="velodyne_to_base" type="fixed">
-      <parent link="base_link" />
-      <child link="velodyne" />
-      <origin xyz="$(arg vlp_xyz)" rpy="$(arg vlp_rpy)"/>
-    </joint>
+    <xacro:VLP-16 name="velodyne" parent="base_link" topic="/sensors/lidar/${vlp_num}/pointcloud">
+      <origin xyz="${vlp_xyz}" rpy="${vlp_rpy}" />
+    </xacro:VLP-16>
   </xacro:macro>
 </robot>

File: urdf/starter_kit.urdf.xacro (robot description, xacro)
@@ -2,14 +2,22 @@
 <robot xmlns:xacro="http://ros.org/wiki/xacro" name="cpr_onav_starter_kit">
   <xacro:macro name="starter_kit" params="name parent starter_kit_xyz starter_kit_rpy ublox_xyz ublox_rpy phidget_spatial_xyz phidget_spatial_rpy d435_xyz d435_rpy rear_d435_xyz rear_d435_rpy">
+    <xacro:include filename="$(find realsense2_description)/urdf/_d435.urdf.xacro" />
     <link name="${name}_link">
       <visual>
         <geometry>
-          <mesh filename="package://cpr_onav_description/meshes/starter_kit.stl" />
+          <mesh filename="package://cpr_onav_description/meshes/starter_kit.stl" scale="0.001 0.001 0.001" />
         </geometry>
+        <material name="yellow" />
+<!--         <material name="yellow" >
+          <color rgba="255 237 4 1" />
+        </material>
+-->
+        <origin xyz="0 0 0" rpy="0 0 0" />
       </visual>
       <collision>
         <geometry>
-          <mesh filename="package://cpr_onav_description/meshes/starter_kit.stl" />
+          <mesh filename="package://cpr_onav_description/meshes/starter_kit.stl" scale="0.001 0.001 0.001" />
         </geometry>
+        <origin xyz="0 0 0" rpy="0 0 0 " />
       </collision>
     </link>
@@ -20,5 +28,21 @@
     </joint>
     <!-- Position GNSS (Ublox) -->
-    <link name="gps_position_link"/>
+    <link name="gps_position_link">
+      <visual>
+        <geometry>
+          <mesh filename="package://cpr_onav_description/meshes/gnss_antenna.stl" />
+        </geometry>
+        <origin xyz="0 0 0" rpy="0 0 0" />
+        <material name="white">
+          <color rgba="1 1 1 1" />
+        </material>
+      </visual>
+      <collision>
+        <geometry>
+          <mesh filename="package://cpr_onav_description/meshes/gnss_antenna.stl" />
+        </geometry>
+        <origin xyz="0 0 0" rpy="0 0 0 " />
+      </collision>
+    </link>
     <joint name="gps_position_to_kit" type="fixed">
       <parent link="${name}_link" />
@@ -34,17 +58,11 @@
     </joint>
     <!-- Realsense D435 -->
-    <link name="front_d435_link"/>
-    <joint name="front_d435_to_kit" type="fixed">
-      <parent link="${name}_link" />
-      <child link="front_d435_link" />
+    <xacro:sensor_d435 name="front_d435" parent="${name}_link" use_mesh="true">
       <origin xyz="${d435_xyz}" rpy="${d435_rpy}"/>
-    </joint>
+    </xacro:sensor_d435>
     <!-- Rear Realsense D435 -->
-    <link name="rear_d435_link"/>
-    <joint name="rear_d435_to_kit" type="fixed">
-      <parent link="${name}_link" />
-      <child link="rear_d435_link" />
+    <xacro:sensor_d435 name="rear_d435" parent="${name}_link" use_mesh="true">
       <origin xyz="${rear_d435_xyz}" rpy="${rear_d435_rpy}"/>
-    </joint>
+    </xacro:sensor_d435>
   </xacro:macro>
 </robot>

Commit message: added charge receiver link

File: urdf/outdoornav_description.urdf.xacro (robot description, xacro)
@@ -58,4 +58,6 @@
     <xacro:arg name="rear_d435_rpy"            default="$(optenv REAR_D435_RPY 0.0 0.0 0.0)" />
     <xacro:arg name="onav_urdf_extras"         default="$(optenv OUTDOORNAV_URDF_EXTRAS empty.urdf)" />
+    <xacro:arg name="enable_docking"           default="$(optenv OUTDOORNAV_ENABLE_DOCKING false)" />
+    <xacro:arg name="charge_receiver_xyz"      default="$(optenv CHARGE_RECEIVER_XYZ 0.0 0.0 0.0)" />
     <!-- Starter Kit -->
     <xacro:if value="${outdoornav_configuration == 'starter'}">
@@ -204,4 +206,12 @@
       <xacro:include filename="$(arg onav_urdf_extras)" />
     </xacro:if>
+    <xacro:if value="$(arg enable_docking)">
+        <link name="charger_link"/>
+        <joint name="charger_to_base" type="fixed">
+          <parent link="base_link" />
+          <child link="charger_link" />
+          <origin xyz="$(arg charge_receiver_xyz)" rpy="0.0 0.0 0.0"/>
+        </joint>
+    </xacro:if>
   </xacro:macro>
 </robot>
