Commit message: modified sensor topic names. and move laser out of block as a temp fix

File: urdf/outdoornav_description.urdf.xacro (robot description, xacro)
@@ -91,10 +91,10 @@
       </xacro:standard_kit>
     </xacro:if>
+    <xacro:include filename="$(find velodyne_description)/urdf/VLP-16.urdf.xacro"/>
+    <xacro:include filename="$(find cpr_onav_description)/urdf/accessories/hokuyo_ust10.urdf.xacro" />
+    <xacro:include filename="$(find cpr_onav_description)/urdf/accessories/sick_lms1xx_mount.urdf.xacro"/>
+    <xacro:include filename="$(find realsense2_description)/urdf/_d435.urdf.xacro" />
     <!-- Custom configuration -->
     <xacro:if value="${outdoornav_configuration == 'custom'}">
-      <xacro:include filename="$(find velodyne_description)/urdf/VLP-16.urdf.xacro"/>
-      <xacro:include filename="$(find cpr_onav_description)/urdf/accessories/hokuyo_ust10.urdf.xacro" />
-      <xacro:include filename="$(find cpr_onav_description)/urdf/accessories/sick_lms1xx_mount.urdf.xacro"/>
-      <xacro:include filename="$(find realsense2_description)/urdf/_d435.urdf.xacro" />
       <!-- Position GPS (Duro) -->
       <xacro:if value="$(arg swiftnav_position_enable)">
@@ -144,5 +144,5 @@
       <!-- Velodyne Link -->
       <xacro:if value="$(arg vlp_enable)">
-        <xacro:VLP-16 name="velodyne" parent="base_link" topic="/sensors/lidar/$(arg vlp_num)/pointcloud">
+        <xacro:VLP-16 name="velodyne" parent="base_link" topic="/sensors/lidar_$(arg vlp_num)/pointcloud">
           <origin xyz="$(arg vlp_xyz)" rpy="$(arg vlp_rpy)" />
         </xacro:VLP-16>
@@ -150,16 +150,11 @@
       <!-- Rear Velodyne Link -->
       <xacro:if value="$(arg rear_vlp_enable)">
-        <xacro:VLP-16 name="rear_velodyne" parent="base_link" topic="/sensors/lidar/$(arg vlp_num)/pointcloud">
+        <xacro:VLP-16 name="rear_velodyne" parent="base_link" topic="/sensors/lidar_$(arg vlp_num)/pointcloud">
           <origin xyz="$(arg rear_vlp_xyz)" rpy="$(arg rear_vlp_rpy)" />
         </xacro:VLP-16>
       </xacro:if>
       <!-- 2D LiDAR(s) Link -->
-      <xacro:if value="$(arg lms1xx_enable)">
-        <xacro:sick_lms1xx_mount prefix="front" parent="base_link" topic="/sensors/lidar/$(arg lms1xx_num)/scan" tower="0" robot_namespace="/">
-          <origin xyz="$(arg lms1xx_xyz)" rpy="$(arg lms1xx_rpy)"/>
-        </xacro:sick_lms1xx_mount>
-      </xacro:if>
       <xacro:if value="$(arg hokuyo_enable)">
-        <xacro:hokuyo_ust10_mount prefix="front_laser" parent_link="base_link" topic="/sensors/lidar/$(arg hokuyo_num)/scan">
+        <xacro:hokuyo_ust10_mount prefix="front_laser" parent_link="base_link" topic="/sensors/lidar_$(arg hokuyo_num)/scan">
             <origin xyz="$(arg hokuyo_xyz)" rpy="$(arg hokuyo_rpy)" />
         </xacro:hokuyo_ust10_mount>
@@ -175,10 +170,10 @@
       <!-- Rear 2D LiDAR(s) Link -->
       <xacro:if value="$(arg rear_lms1xx_enable)">
-        <xacro:sick_lms1xx_mount prefix="rear" parent="base_link" topic="/sensors/lidar/$(arg rear_lms1xx_num)/scan" tower="0" robot_namespace="/">
+        <xacro:sick_lms1xx_mount prefix="rear" parent="base_link" topic="/sensors/lidar_$(arg rear_lms1xx_num)/scan" tower="0" robot_namespace="/">
           <origin xyz="$(arg lms1xx_xyz)" rpy="$(arg lms1xx_rpy)"/>
         </xacro:sick_lms1xx_mount>
       </xacro:if>
       <xacro:if value="$(arg rear_hokuyo_enable)">
-        <xacro:hokuyo_ust10_mount prefix="rear_laser" parent_link="base_link" topic="/sensors/lidar/$(arg rear_hokuyo_num)/scan">
+        <xacro:hokuyo_ust10_mount prefix="rear_laser" parent_link="base_link" topic="/sensors/lidar_$(arg rear_hokuyo_num)/scan">
             <origin xyz="$(arg hokuyo_xyz)" rpy="$(arg hokuyo_rpy)" />
         </xacro:hokuyo_ust10_mount>
@@ -206,4 +201,9 @@
       <xacro:include filename="$(arg onav_urdf_extras)" />
     </xacro:if>
+    <xacro:if value="$(arg lms1xx_enable)">
+      <xacro:sick_lms1xx_mount prefix="front" parent="base_link" topic="/sensors/lidar_$(arg lms1xx_num)/scan" tower="0" robot_namespace="/">
+        <origin xyz="$(arg lms1xx_xyz)" rpy="$(arg lms1xx_rpy)"/>
+      </xacro:sick_lms1xx_mount>
+    </xacro:if>
     <xacro:if value="$(arg enable_docking)">
         <link name="charger_link"/>

File: urdf/standard_kit.urdf.xacro (robot description, xacro)
@@ -57,5 +57,5 @@
     </joint>
     <!-- Velodyne Link -->
-    <xacro:VLP-16 name="velodyne" parent="base_link" topic="/sensors/lidar/${vlp_num}/pointcloud">
+    <xacro:VLP-16 name="velodyne" parent="base_link" topic="/sensors/lidar_${vlp_num}/pointcloud">
       <origin xyz="${vlp_xyz}" rpy="${vlp_rpy}" />
     </xacro:VLP-16>

Commit message: fix: move lms1xx link back into correct location. this bug was resolve in the intall script. update hokuyo prefix

File: urdf/outdoornav_description.urdf.xacro (robot description, xacro)
@@ -155,6 +155,11 @@
       </xacro:if>
       <!-- 2D LiDAR(s) Link -->
+      <xacro:if value="$(arg lms1xx_enable)">
+        <xacro:sick_lms1xx_mount prefix="front" parent="base_link" topic="/sensors/lidar_$(arg lms1xx_num)/scan" tower="0" robot_namespace="/">
+          <origin xyz="$(arg lms1xx_xyz)" rpy="$(arg lms1xx_rpy)"/>
+        </xacro:sick_lms1xx_mount>
+      </xacro:if>
       <xacro:if value="$(arg hokuyo_enable)">
-        <xacro:hokuyo_ust10_mount prefix="front_laser" parent_link="base_link" topic="/sensors/lidar_$(arg hokuyo_num)/scan">
+        <xacro:hokuyo_ust10_mount prefix="front" parent_link="base_link" topic="/sensors/lidar_$(arg hokuyo_num)/scan">
             <origin xyz="$(arg hokuyo_xyz)" rpy="$(arg hokuyo_rpy)" />
         </xacro:hokuyo_ust10_mount>
@@ -175,5 +180,5 @@
       </xacro:if>
       <xacro:if value="$(arg rear_hokuyo_enable)">
-        <xacro:hokuyo_ust10_mount prefix="rear_laser" parent_link="base_link" topic="/sensors/lidar_$(arg rear_hokuyo_num)/scan">
+        <xacro:hokuyo_ust10_mount prefix="rear" parent_link="base_link" topic="/sensors/lidar_$(arg rear_hokuyo_num)/scan">
             <origin xyz="$(arg hokuyo_xyz)" rpy="$(arg hokuyo_rpy)" />
         </xacro:hokuyo_ust10_mount>
@@ -201,9 +206,4 @@
       <xacro:include filename="$(arg onav_urdf_extras)" />
     </xacro:if>
-    <xacro:if value="$(arg lms1xx_enable)">
-      <xacro:sick_lms1xx_mount prefix="front" parent="base_link" topic="/sensors/lidar_$(arg lms1xx_num)/scan" tower="0" robot_namespace="/">
-        <origin xyz="$(arg lms1xx_xyz)" rpy="$(arg lms1xx_rpy)"/>
-      </xacro:sick_lms1xx_mount>
-    </xacro:if>
     <xacro:if value="$(arg enable_docking)">
         <link name="charger_link"/>

Commit message: Add Husky Observer backpack model, Q62 meshes, support for `observer` configuration

File: urdf/outdoornav_description.urdf.xacro (robot description, xacro)
@@ -54,7 +54,13 @@
     <xacro:arg name="d435_xyz"                 default="$(optenv D435_XYZ 0.0 0.0 0.0)" />
     <xacro:arg name="d435_rpy"                 default="$(optenv D435_RPY 0.0 0.0 0.0)" />
+    <xacro:arg name="d435_num"                 default="$(optenv D435_NUM 0)" />
     <xacro:arg name="rear_d435_enable"         default="$(optenv REAR_D435_ENABLE_DRIVER false)" />
     <xacro:arg name="rear_d435_xyz"            default="$(optenv REAR_D435_XYZ 0.0 0.0 0.0)" />
     <xacro:arg name="rear_d435_rpy"            default="$(optenv REAR_D435_RPY 0.0 0.0 0.0)" />
+    <xacro:arg name="rear_d435_num"            default="$(optenv REAR_D435_NUM 1)" />
+    <xacro:arg name="axis_ptz_enable"          default="$(optenv AXIS_PTZ_ENABLE_DRIVER false)" />
+    <xacro:arg name="axis_ptz_num"             default="$(optenv AXIS_PTZ_NUM 0)" />
+    <xacro:arg name="axis_q62_xyz"             default="$(optenv AXIS_Q62_XYZ 0 0 0)" />
+    <xacro:arg name="axis_q62_rpy"             default="$(optenv AXIS_Q62_RPY 0 0 0)" />
     <xacro:arg name="onav_urdf_extras"         default="$(optenv OUTDOORNAV_URDF_EXTRAS empty.urdf)" />
     <xacro:arg name="enable_docking"           default="$(optenv OUTDOORNAV_ENABLE_DOCKING false)" />
@@ -91,4 +97,62 @@
       </xacro:standard_kit>
     </xacro:if>
+    <!-- Husky Observer configuration -->
+    <xacro:if value="${outdoornav_configuration == 'observer'}">
+      <xacro:include filename="$(find velodyne_description)/urdf/VLP-16.urdf.xacro"/>
+      <xacro:include filename="$(find cpr_onav_description)/urdf/accessories/hokuyo_ust10.urdf.xacro" />
+      <xacro:include filename="$(find cpr_onav_description)/urdf/accessories/sick_lms1xx_mount.urdf.xacro"/>
+      <xacro:include filename="$(find realsense2_description)/urdf/_d435.urdf.xacro" />
+      <xacro:include filename="$(find cpr_onav_description)/urdf/accessories/d435_gazebo.urdf.xacro" />
+      <xacro:include filename="$(find cpr_onav_description)/urdf/accessories/axis_q62.urdf.xacro" />
+      <!-- Main backpack shell & mast assembly -->
+      <xacro:include filename="$(find cpr_onav_description)/urdf/husky_observer.urdf.xacro" />
+      <!-- Position GPS (Duro) -->
+      <link name="gps_position_link"/>
+      <joint name="gps_position_to_base" type="fixed">
+        <parent link="base_link" />
+        <child link="gps_position_link" />
+        <origin xyz="$(arg swiftnav_position_xyz)" rpy="$(arg swiftnav_position_rpy)"/>
+      </joint>
+      <!-- Heading GPS -->
+      <link name="gps_heading_link"/>
+      <joint name="gps_heading_to_base" type="fixed">
+        <parent link="base_link" />
+        <child link="gps_heading_link" />
+        <origin xyz="$(arg swiftnav_heading_xyz)" rpy="$(arg swiftnav_heading_rpy)"/>
+      </joint>
+      <!-- Microstrain Link -->
+      <link name="microstrain_link"/>
+      <joint name="microstrain_to_base" type="fixed">
+        <parent link="base_link" />
+        <child link="microstrain_link" />
+        <origin xyz="$(arg microstrain_xyz)" rpy="$(arg microstrain_rpy)"/>
+      </joint>
+      <!-- Velodyne Link -->
+      <xacro:VLP-16 name="velodyne" parent="base_link" topic="/sensors/lidar_$(arg vlp_num)/pointcloud">
+        <origin xyz="$(arg vlp_xyz)" rpy="$(arg vlp_rpy)" />
+      </xacro:VLP-16>
+      <!-- 2D LiDAR(s) Link -->
+      <xacro:hokuyo_ust10_mount prefix="front" parent_link="base_link" topic="/sensors/lidar_$(arg hokuyo_num)/scan">
+          <origin xyz="$(arg hokuyo_xyz)" rpy="$(arg hokuyo_rpy)" />
+      </xacro:hokuyo_ust10_mount>
+      <xacro:if value="$(arg rear_hokuyo_enable)">
+        <xacro:hokuyo_ust10_mount prefix="rear" parent_link="base_link" topic="/sensors/lidar_$(arg rear_hokuyo_num)/scan">
+            <origin xyz="$(arg hokuyo_xyz)" rpy="$(arg hokuyo_rpy)" />
+        </xacro:hokuyo_ust10_mount>
+      </xacro:if>
+      <!-- Realsense D435 Link -->
+      <xacro:sensor_d435 name="front_d435" parent="base_link" use_mesh="true">
+        <origin xyz="$(arg d435_xyz)" rpy="$(arg d435_rpy)"/>
+      </xacro:sensor_d435>
+      <xacro:d435_gazebo name="front_d435" topic_n="$(arg d435_num)" />
+      <xacro:sensor_d435 name="rear_d435" parent="base_link" use_mesh="true">
+        <origin xyz="$(arg rear_d435_xyz)" rpy="$(arg rear_d435_rpy)"/>
+      </xacro:sensor_d435>
+      <xacro:d435_gazebo name="rear_d435" topic_n="$(arg rear_d435_num)" />
+      <!-- Axis Q62 PTZ camera -->
+      <xacro:axis_q62 prefix="ptz_camera" parent="base_link" axis_ptz_num="$(arg axis_ptz_num)">
+        <origin xyz="$(arg axis_q62_xyz)" rpy="$(arg axis_q62_rpy)" />
+      </xacro:axis_q62>
+    </xacro:if>
     <!-- Custom configuration -->
     <xacro:if value="${outdoornav_configuration == 'custom'}">
@@ -97,4 +161,6 @@
       <xacro:include filename="$(find cpr_onav_description)/urdf/accessories/sick_lms1xx_mount.urdf.xacro"/>
       <xacro:include filename="$(find realsense2_description)/urdf/_d435.urdf.xacro" />
+      <xacro:include filename="$(find cpr_onav_description)/urdf/accessories/d435_gazebo.urdf.xacro" />
+      <xacro:include filename="$(find cpr_onav_description)/urdf/accessories/axis_q62.urdf.xacro" />
       <!-- Position GPS (Duro) -->
       <xacro:if value="$(arg swiftnav_position_enable)">
@@ -197,4 +263,5 @@
           <origin xyz="$(arg d435_xyz)" rpy="$(arg d435_rpy)"/>
         </xacro:sensor_d435>
+        <xacro:d435_gazebo name="front_d435" topic_n="$(arg d435_num)" />
       </xacro:if>
       <xacro:if value="$(arg rear_d435_enable)">
@@ -202,4 +269,11 @@
           <origin xyz="$(arg rear_d435_xyz)" rpy="$(arg rear_d435_rpy)"/>
         </xacro:sensor_d435>
+        <xacro:d435_gazebo name="rear_d435" topic_n="$(arg rear_d435_num)" />
+      </xacro:if>
+      <!-- Axis Q62 PTZ camera -->
+      <xacro:if value="$(arg axis_ptz_enable)">
+        <xacro:axis_q62 prefix="ptz_camera" parent="base_link" axis_ptz_num="$(arg axis_ptz_num)">
+          <origin xyz="$(arg axis_q62_xyz)" rpy="$(arg axis_q62_rpy)" />
+        </xacro:axis_q62>
       </xacro:if>
       <!-- Optional for OEM platforms or additional sensors customers want to use as inputs to OutdoorNav -->

Commit message: Add a new macro for the GNSS antennas, including collision bodies

File: urdf/outdoornav_description.urdf.xacro (robot description, xacro)
@@ -105,20 +105,15 @@
       <xacro:include filename="$(find cpr_onav_description)/urdf/accessories/d435_gazebo.urdf.xacro" />
       <xacro:include filename="$(find cpr_onav_description)/urdf/accessories/axis_q62.urdf.xacro" />
+      <xacro:include filename="$(find cpr_onav_description)/urdf/accessories/gnss_antenna.urdf.xacro" />
       <!-- Main backpack shell & mast assembly -->
       <xacro:include filename="$(find cpr_onav_description)/urdf/husky_observer.urdf.xacro" />
       <!-- Position GPS (Duro) -->
-      <link name="gps_position_link"/>
-      <joint name="gps_position_to_base" type="fixed">
-        <parent link="base_link" />
-        <child link="gps_position_link" />
+      <xacro:gnss_antenna name="gps_position" parent="base_link" gps_num="0">
         <origin xyz="$(arg swiftnav_position_xyz)" rpy="$(arg swiftnav_position_rpy)"/>
-      </joint>
+      </xacro:gnss_antenna>
       <!-- Heading GPS -->
-      <link name="gps_heading_link"/>
-      <joint name="gps_heading_to_base" type="fixed">
-        <parent link="base_link" />
-        <child link="gps_heading_link" />
+      <xacro:gnss_antenna name="gps_heading" parent="base_link" gps_num="1">
         <origin xyz="$(arg swiftnav_heading_xyz)" rpy="$(arg swiftnav_heading_rpy)"/>
-      </joint>
+      </xacro:gnss_antenna>
       <!-- Microstrain Link -->
       <link name="microstrain_link"/>

Commit message: Fix the position of the rear lidar

File: urdf/outdoornav_description.urdf.xacro (robot description, xacro)
@@ -133,5 +133,5 @@
       <xacro:if value="$(arg rear_hokuyo_enable)">
         <xacro:hokuyo_ust10_mount prefix="rear" parent_link="base_link" topic="/sensors/lidar_$(arg rear_hokuyo_num)/scan">
-            <origin xyz="$(arg hokuyo_xyz)" rpy="$(arg hokuyo_rpy)" />
+            <origin xyz="$(arg rear_hokuyo_xyz)" rpy="$(arg rear_hokuyo_rpy)" />
         </xacro:hokuyo_ust10_mount>
       </xacro:if>

Commit message: don't pull in axis q62 meshes for all axis ptz camera integrations

File: urdf/outdoornav_description.urdf.xacro (robot description, xacro)
@@ -60,4 +60,5 @@
     <xacro:arg name="rear_d435_num"            default="$(optenv REAR_D435_NUM 1)" />
     <xacro:arg name="axis_ptz_enable"          default="$(optenv AXIS_PTZ_ENABLE_DRIVER false)" />
+    <xacro:arg name="axis_q62_enable"          default="$(optenv AXIS_Q62_ENABLE false)" />
     <xacro:arg name="axis_ptz_num"             default="$(optenv AXIS_PTZ_NUM 0)" />
     <xacro:arg name="axis_q62_xyz"             default="$(optenv AXIS_Q62_XYZ 0 0 0)" />
@@ -268,7 +269,9 @@
       <!-- Axis Q62 PTZ camera -->
       <xacro:if value="$(arg axis_ptz_enable)">
-        <xacro:axis_q62 prefix="ptz_camera" parent="base_link" axis_ptz_num="$(arg axis_ptz_num)">
-          <origin xyz="$(arg axis_q62_xyz)" rpy="$(arg axis_q62_rpy)" />
-        </xacro:axis_q62>
+        <xacro:if value="$(arg axis_q62_enable)">
+          <xacro:axis_q62 prefix="ptz_camera" parent="base_link" axis_ptz_num="$(arg axis_ptz_num)">
+            <origin xyz="$(arg axis_q62_xyz)" rpy="$(arg axis_q62_rpy)" />
+          </xacro:axis_q62>
+        </xacro:if>
       </xacro:if>
       <!-- Optional for OEM platforms or additional sensors customers want to use as inputs to OutdoorNav -->

Commit message: Add: Custom 3d_lidar.urdf.xacro for simulating VLP16 / 3d lidars
Signed-off-by: Stephen Phillips <stphillips@clearpathrobotics.com>

File: urdf/outdoornav_description.urdf.xacro (robot description, xacro)
@@ -124,8 +124,34 @@
         <origin xyz="$(arg microstrain_xyz)" rpy="$(arg microstrain_rpy)"/>
       </joint>
-      <!-- Velodyne Link -->
-      <xacro:VLP-16 name="velodyne" parent="base_link" topic="/sensors/lidar_$(arg vlp_num)/pointcloud">
-        <origin xyz="$(arg vlp_xyz)" rpy="$(arg vlp_rpy)" />
-      </xacro:VLP-16>
+      <!--
+          Velodyne VLP-16 in the tower
+          The 3D lidar can be a CPU hog, especially in Docker where GPU support can't be used. Therefore we expose
+          a lot of the low-level lidar parameters so we can fine-tune the lidar's performance if needed
+          Settings that are different from the VLP-16 defaults are noted with a comment. Other settings are unchanged.
+        -->
+      <xacro:property name="vertical_scan_min_h_angle" value="$(optenv CPR_SIMULATION_3D_LIDAR_MIN_H_ANGLE -3.1415926535897931)" />
+      <xacro:property name="vertical_scan_max_h_angle" value="$(optenv CPR_SIMULATION_3D_LIDAR_MAX_H_ANGLE  3.1415926535897931)" />
+      <xacro:property name="vertical_scan_min_v_angle" value="$(optenv CPR_SIMULATION_3D_LIDAR_MIN_V_ANGLE -0.2617993877991494)" />
+      <xacro:property name="vertical_scan_max_v_angle" value="$(optenv CPR_SIMULATION_3D_LIDAR_MAX_V_ANGLE  0.2617993877991494)" />
+      <xacro:property name="num_samples"               value="$(optenv CPR_SIMULATION_3D_LIDAR_SAMPLES      720)" />  <!-- VLP-16 default: 1875 -->
+      <xacro:property name="num_rings"                 value="$(optenv CPR_SIMULATION_3D_LIDAR_RINGS        8)" />    <!-- VLP-16 default: 16 -->
+      <xacro:property name="resolution"                value="$(optenv CPR_SIMULATION_3D_LIDAR_RESOLUTION   0.01)" /> <!-- VLP-16 default: 0.001 -->
+      <xacro:property name="lidar_hz"                  value="$(optenv CPR_SIMULATION_3D_LIDAR_HZ           5)" />    <!-- VLP-16 default: 10 -->
+      <xacro:property name="enable_gpu"                value="$(optenv CPR_SIMULATION_3D_LIDAR_ENABLE_GPU   false)" />
+      <xacro:include filename="$(find cpr_onav_description)/urdf/accessories/3d_lidar.urdf.xacro" />
+      <xacro:if value="$(optenv CPR_SIMULATION_ENABLE_3D_LIDAR 1)">
+        <xacro:custom_velodyne name="velodyne" parent="base_link" topic="/sensors/lidar_$(arg vlp_num)/pointcloud"
+                               min_v_angle="${vertical_scan_min_v_angle}"
+                               max_v_angle="${vertical_scan_max_v_angle}"
+                               min_h_angle="${vertical_scan_min_h_angle}"
+                               max_h_angle="${vertical_scan_max_h_angle}"
+                               resolution="${resolution}"
+                               hz="${lidar_hz}"
+                               lasers="${num_rings}"
+                               samples="${num_samples}"
+                               gpu="${enable_gpu}">
+          <origin xyz="$(arg vlp_xyz)" rpy="$(arg vlp_rpy)" />
+        </xacro:custom_velodyne>
+      </xacro:if>
       <!-- 2D LiDAR(s) Link -->
       <xacro:hokuyo_ust10_mount prefix="front" parent_link="base_link" topic="/sensors/lidar_$(arg hokuyo_num)/scan">

Commit message: added xvn link to urdf

File: urdf/outdoornav_description.urdf.xacro (robot description, xacro)
@@ -64,4 +64,7 @@
     <xacro:arg name="axis_q62_xyz"             default="$(optenv AXIS_Q62_XYZ 0 0 0)" />
     <xacro:arg name="axis_q62_rpy"             default="$(optenv AXIS_Q62_RPY 0 0 0)" />
+    <xacro:arg name="xvn_enable"               default="$(optenv XVN_ENABLE_DRIVER false)" />
+    <xacro:arg name="xvn_xyz"                  default="$(optenv XVN_XYZ 0 0 0)" />
+    <xacro:arg name="xvn_rpy"                  default="$(optenv XVN_RPY 0 0 0)" />
     <xacro:arg name="onav_urdf_extras"         default="$(optenv OUTDOORNAV_URDF_EXTRAS empty.urdf)" />
     <xacro:arg name="enable_docking"           default="$(optenv OUTDOORNAV_ENABLE_DOCKING false)" />
@@ -212,4 +215,12 @@
         </joint>
       </xacro:if>
+      <xacro:if value="$(arg xvn_enable)">
+        <link name="xvn_link"/>
+        <joint name="xvn_to_base" type="fixed">
+          <parent link="base_link" />
+          <child link="xvn_link" />
+          <origin xyz="$(arg xvn_xyz)" rpy="$(arg xvn_rpy)"/>
+        </joint>
+      </xacro:if>
       <!-- Microstrain Link -->
       <xacro:if value="$(arg microstrain_enable)">

Commit message: fix rear laser xyz, rpy

File: urdf/outdoornav_description.urdf.xacro (robot description, xacro)
@@ -275,10 +275,10 @@
       <xacro:if value="$(arg rear_lms1xx_enable)">
         <xacro:sick_lms1xx_mount prefix="rear" parent="base_link" topic="/sensors/lidar_$(arg rear_lms1xx_num)/scan" tower="0" robot_namespace="/">
-          <origin xyz="$(arg lms1xx_xyz)" rpy="$(arg lms1xx_rpy)"/>
+          <origin xyz="$(arg rear_lms1xx_xyz)" rpy="$(arg rear_lms1xx_rpy)"/>
         </xacro:sick_lms1xx_mount>
       </xacro:if>
       <xacro:if value="$(arg rear_hokuyo_enable)">
         <xacro:hokuyo_ust10_mount prefix="rear" parent_link="base_link" topic="/sensors/lidar_$(arg rear_hokuyo_num)/scan">
-            <origin xyz="$(arg hokuyo_xyz)" rpy="$(arg hokuyo_rpy)" />
+            <origin xyz="$(arg rear_hokuyo_xyz)" rpy="$(arg rear_hokuyo_rpy)" />
         </xacro:hokuyo_ust10_mount>
       </xacro:if>
