Commit message: add dependency on jackal fenders

File: urdf/outdoornav_description.urdf.xacro (robot description, xacro)
@@ -2,4 +2,6 @@
 <robot xmlns:xacro="http://ros.org/wiki/xacro" name="outdoornav_sensors">
   <xacro:macro name="outdoornav_sensors" params="outdoornav_configuration">
+    <xacro:arg name="jackal_front_fender"      default="$(optenv JACKAL_FRONT_ACCESSORY_FENDER false)" />
+    <xacro:arg name="jackal_rear_fender"       default="$(optenv JACKAL_REAR_ACCESSORY_FENDER false)" />
     <xacro:arg name="starter_kit_xyz"          default="$(optenv STARTER_KIT_XYZ 0.0 0.0 0.0)" />
     <xacro:arg name="starter_kit_rpy"          default="$(optenv STARTER_KIT_RPY 0.0 0.0 0.0)" />
@@ -260,7 +262,14 @@
       </xacro:if>
       <xacro:if value="$(arg hokuyo_enable)">
-        <xacro:hokuyo_ust10_mount prefix="front" parent_link="base_link" topic="/sensors/lidar_$(arg hokuyo_num)/scan">
-            <origin xyz="$(arg hokuyo_xyz)" rpy="$(arg hokuyo_rpy)" />
-        </xacro:hokuyo_ust10_mount>
+        <xacro:if value="$(arg jackal_front_fender)">
+          <xacro:hokuyo_ust10_mount prefix="front" parent_link="front_fender_accessory_link" topic="/sensors/lidar_$(arg hokuyo_num)/scan">
+              <origin xyz="$(arg hokuyo_xyz)" rpy="$(arg hokuyo_rpy)" />
+          </xacro:hokuyo_ust10_mount>
+        </xacro:if>
+        <xacro:unless value="$(arg jackal_front_fender)">
+          <xacro:hokuyo_ust10_mount prefix="front" parent_link="base_link" topic="/sensors/lidar_$(arg hokuyo_num)/scan">
+              <origin xyz="$(arg hokuyo_xyz)" rpy="$(arg hokuyo_rpy)" />
+          </xacro:hokuyo_ust10_mount>
+        </xacro:if>
       </xacro:if>
       <xacro:if value="$(arg outdoorscan_enable)">
@@ -279,7 +288,14 @@
       </xacro:if>
       <xacro:if value="$(arg rear_hokuyo_enable)">
-        <xacro:hokuyo_ust10_mount prefix="rear" parent_link="base_link" topic="/sensors/lidar_$(arg rear_hokuyo_num)/scan">
-            <origin xyz="$(arg rear_hokuyo_xyz)" rpy="$(arg rear_hokuyo_rpy)" />
-        </xacro:hokuyo_ust10_mount>
+        <xacro:if value="$(arg jackal_rear_fender)">
+          <xacro:hokuyo_ust10_mount prefix="rear" parent_link="rear_fender_accessory_link" topic="/sensors/lidar_$(arg rear_hokuyo_num)/scan">
+              <origin xyz="$(arg rear_hokuyo_xyz)" rpy="$(arg rear_hokuyo_rpy)" />
+          </xacro:hokuyo_ust10_mount>
+        </xacro:if>
+        <xacro:unless value="$(arg jackal_rear_fender)">
+          <xacro:hokuyo_ust10_mount prefix="rear" parent_link="base_link" topic="/sensors/lidar_$(arg rear_hokuyo_num)/scan">
+              <origin xyz="$(arg rear_hokuyo_xyz)" rpy="$(arg rear_hokuyo_rpy)" />
+          </xacro:hokuyo_ust10_mount>
+        </xacro:if>
       </xacro:if>
       <xacro:if value="$(arg rear_outdoorscan_enable)">

Commit message: revert fender fix. use position relative to base_link

File: urdf/outdoornav_description.urdf.xacro (robot description, xacro)
@@ -262,14 +262,7 @@
       </xacro:if>
       <xacro:if value="$(arg hokuyo_enable)">
-        <xacro:if value="$(arg jackal_front_fender)">
-          <xacro:hokuyo_ust10_mount prefix="front" parent_link="front_fender_accessory_link" topic="/sensors/lidar_$(arg hokuyo_num)/scan">
-              <origin xyz="$(arg hokuyo_xyz)" rpy="$(arg hokuyo_rpy)" />
-          </xacro:hokuyo_ust10_mount>
-        </xacro:if>
-        <xacro:unless value="$(arg jackal_front_fender)">
-          <xacro:hokuyo_ust10_mount prefix="front" parent_link="base_link" topic="/sensors/lidar_$(arg hokuyo_num)/scan">
-              <origin xyz="$(arg hokuyo_xyz)" rpy="$(arg hokuyo_rpy)" />
-          </xacro:hokuyo_ust10_mount>
-        </xacro:unless>
+        <xacro:hokuyo_ust10_mount prefix="front" parent_link="base_link" topic="/sensors/lidar_$(arg hokuyo_num)/scan">
+          <origin xyz="$(arg hokuyo_xyz)" rpy="$(arg hokuyo_rpy)" />
+        </xacro:hokuyo_ust10_mount>
       </xacro:if>
       <xacro:if value="$(arg outdoorscan_enable)">
@@ -288,14 +281,7 @@
       </xacro:if>
       <xacro:if value="$(arg rear_hokuyo_enable)">
-        <xacro:if value="$(arg jackal_rear_fender)">
-          <xacro:hokuyo_ust10_mount prefix="rear" parent_link="rear_fender_accessory_link" topic="/sensors/lidar_$(arg rear_hokuyo_num)/scan">
-              <origin xyz="$(arg rear_hokuyo_xyz)" rpy="$(arg rear_hokuyo_rpy)" />
-          </xacro:hokuyo_ust10_mount>
-        </xacro:if>
-        <xacro:unless value="$(arg jackal_rear_fender)">
-          <xacro:hokuyo_ust10_mount prefix="rear" parent_link="base_link" topic="/sensors/lidar_$(arg rear_hokuyo_num)/scan">
-              <origin xyz="$(arg rear_hokuyo_xyz)" rpy="$(arg rear_hokuyo_rpy)" />
-          </xacro:hokuyo_ust10_mount>
-        </xacro:unless>
+        <xacro:hokuyo_ust10_mount prefix="rear" parent_link="base_link" topic="/sensors/lidar_$(arg rear_hokuyo_num)/scan">
+          <origin xyz="$(arg rear_hokuyo_xyz)" rpy="$(arg rear_hokuyo_rpy)" />
+        </xacro:hokuyo_ust10_mount>
       </xacro:if>
       <xacro:if value="$(arg rear_outdoorscan_enable)">

Commit message: added xvn stl to model

File: urdf/outdoornav_description.urdf.xacro (robot description, xacro)
@@ -218,5 +218,19 @@
       </xacro:if>
       <xacro:if value="$(arg xvn_enable)">
-        <link name="xvn_link"/>
+        <link name="xvn_link">
+          <visual>
+            <geometry>
+              <mesh filename="package://cpr_onav_description/meshes/xvn.stl" scale="0.001 0.001 0.001" />
+            </geometry>
+            <material name="yellow" />
+            <origin xyz="0 0 0" rpy="0 0 0" />
+          </visual>
+          <collision>
+            <geometry>
+              <mesh filename="package://cpr_onav_description/meshes/zvn.stl" scale="0.001 0.001 0.001" />
+            </geometry>
+            <origin xyz="0 0 0" rpy="0 0 0 " />
+          </collision>
+        </link>
         <joint name="xvn_to_base" type="fixed">
           <parent link="base_link" />

Commit message: fix axis of xvn stl file

File: urdf/outdoornav_description.urdf.xacro (robot description, xacro)
@@ -228,5 +228,5 @@
           <collision>
             <geometry>
-              <mesh filename="package://cpr_onav_description/meshes/zvn.stl" scale="0.001 0.001 0.001" />
+              <mesh filename="package://cpr_onav_description/meshes/xvn.stl" scale="0.001 0.001 0.001" />
             </geometry>
             <origin xyz="0 0 0" rpy="0 0 0 " />

Commit message: added color of xvn unit

File: urdf/outdoornav_description.urdf.xacro (robot description, xacro)
@@ -218,4 +218,5 @@
       </xacro:if>
       <xacro:if value="$(arg xvn_enable)">
+        <material name="silver"> <color rgba="${192/255} ${192/255} ${192/255} 1.0"/> </material>
         <link name="xvn_link">
           <visual>
@@ -223,5 +224,5 @@
               <mesh filename="package://cpr_onav_description/meshes/xvn.stl" scale="0.001 0.001 0.001" />
             </geometry>
-            <material name="yellow" />
+            <material name="silver" />
             <origin xyz="0 0 0" rpy="0 0 0" />
           </visual>

Commit message: add ptz camera links to urdf

File: urdf/outdoornav_description.urdf.xacro (robot description, xacro)
@@ -60,8 +60,14 @@
     <xacro:arg name="rear_d435_num"            default="$(optenv REAR_D435_NUM 1)" />
     <xacro:arg name="axis_ptz_enable"          default="$(optenv AXIS_PTZ_ENABLE_DRIVER false)" />
-    <xacro:arg name="axis_q62_enable"          default="$(optenv AXIS_Q62_ENABLE false)" />
+    <xacro:arg name="axis_q62_enable"          default="$(optenv AXIS_PTZ_Q62_ENABLE_DRIVER false)" />
     <xacro:arg name="axis_ptz_num"             default="$(optenv AXIS_PTZ_NUM 0)" />
+    <xacro:arg name="axis_ptz_xyz"             default="$(optenv AXIS_PTZ_XYZ 0 0 0)" />
+    <xacro:arg name="axis_ptz_rpy"             default="$(optenv AXIS_PTZ_RPY 0 0 0)" />
     <xacro:arg name="axis_q62_xyz"             default="$(optenv AXIS_Q62_XYZ 0 0 0)" />
     <xacro:arg name="axis_q62_rpy"             default="$(optenv AXIS_Q62_RPY 0 0 0)" />
+    <xacro:arg name="rear_axis_ptz_enable"     default="$(optenv REAR_AXIS_PTZ_ENABLE_DRIVER false)" />
+    <xacro:arg name="rear_axis_ptz_num"        default="$(optenv REAR_AXIS_PTZ_NUM 0)" />
+    <xacro:arg name="rear_axis_ptz_xyz"        default="$(optenv REAR_AXIS_PTZ_XYZ 0 0 0)" />
+    <xacro:arg name="rear_axis_ptz_rpy"        default="$(optenv REAR_AXIS_PTZ_RPY 0 0 0)" />
     <xacro:arg name="onav_urdf_extras"         default="$(optenv OUTDOORNAV_URDF_EXTRAS empty.urdf)" />
     <xacro:arg name="enable_docking"           default="$(optenv OUTDOORNAV_ENABLE_DOCKING false)" />
@@ -293,11 +299,27 @@
         <xacro:d435_gazebo name="rear_d435" topic_n="$(arg rear_d435_num)" />
       </xacro:if>
+      <!-- Axis PTZ camera -->
+      <xacro:if value="$(arg axis_ptz_enable)">
+        <link name="axis_ptz_camera_link"/>
+        <joint name="axis_to_base" type="fixed">
+          <parent link="base_link" />
+          <child link="axis_ptz_camera_link" />
+          <origin xyz="$(arg axis_ptz_xyz)" rpy="$(arg axis_ptz_rpy)"/>
+        </joint>
+      </xacro:if>
+      <!-- Rear Axis PTZ camera -->
+      <xacro:if value="$(arg rear_axis_ptz_enable)">
+        <link name="rear_axis_ptz_camera_link"/>
+        <joint name="rear_axis_to_base" type="fixed">
+          <parent link="base_link" />
+          <child link="rear_axis_ptz_camera_link" />
+          <origin xyz="$(arg rear_axis_ptz_xyz)" rpy="$(arg rear_axis_ptz_rpy)"/>
+        </joint>
+      </xacro:if>
       <!-- Axis Q62 PTZ camera -->
-      <xacro:if value="$(arg axis_ptz_enable)">
-        <xacro:if value="$(arg axis_q62_enable)">
-          <xacro:axis_q62 prefix="ptz_camera" parent="base_link" axis_ptz_num="$(arg axis_ptz_num)">
-            <origin xyz="$(arg axis_q62_xyz)" rpy="$(arg axis_q62_rpy)" />
-          </xacro:axis_q62>
-        </xacro:if>
+      <xacro:if value="$(arg axis_q62_enable)">
+        <xacro:axis_q62 prefix="ptz_camera" parent="base_link" axis_ptz_num="$(arg axis_ptz_num)">
+          <origin xyz="$(arg axis_q62_xyz)" rpy="$(arg axis_q62_rpy)" />
+        </xacro:axis_q62>
       </xacro:if>
       <!-- Optional for OEM platforms or additional sensors customers want to use as inputs to OutdoorNav -->

Commit message: Use the axis_description package for the camera URDFs, add axis dome camera meshes

File: urdf/outdoornav_description.urdf.xacro (robot description, xacro)
@@ -111,5 +111,5 @@
       <xacro:include filename="$(find realsense2_description)/urdf/_d435.urdf.xacro" />
       <xacro:include filename="$(find cpr_onav_description)/urdf/accessories/d435_gazebo.urdf.xacro" />
-      <xacro:include filename="$(find cpr_onav_description)/urdf/accessories/axis_q62.urdf.xacro" />
+      <xacro:include filename="$(find axis_description)/urdf/axis_q62.urdf.xacro" />
       <xacro:include filename="$(find cpr_onav_description)/urdf/accessories/gnss_antenna.urdf.xacro" />
       <!-- Main backpack shell & mast assembly -->
@@ -190,5 +190,7 @@
       <xacro:include filename="$(find realsense2_description)/urdf/_d435.urdf.xacro" />
       <xacro:include filename="$(find cpr_onav_description)/urdf/accessories/d435_gazebo.urdf.xacro" />
-      <xacro:include filename="$(find cpr_onav_description)/urdf/accessories/axis_q62.urdf.xacro" />
+      <xacro:include filename="$(find axis_description)/urdf/axis_dome_fixed.urdf.xacro" />
+      <xacro:include filename="$(find axis_description)/urdf/axis_dome_ptz.urdf.xacro" />
+      <xacro:include filename="$(find axis_description)/urdf/axis_q62.urdf.xacro" />
       <!-- Position GPS (Duro) -->
       <xacro:if value="$(arg swiftnav_position_enable)">
@@ -301,23 +303,17 @@
       <!-- Axis PTZ camera -->
       <xacro:if value="$(arg axis_ptz_enable)">
-        <link name="axis_ptz_camera_link"/>
-        <joint name="axis_to_base" type="fixed">
-          <parent link="base_link" />
-          <child link="axis_ptz_camera_link" />
+        <xacro:axis_dome_ptz prefix="axis_ptz_camera" parent="base_link" topic="/sensors/camera_$(arg axis_ptz_num)/image_raw">
           <origin xyz="$(arg axis_ptz_xyz)" rpy="$(arg axis_ptz_rpy)"/>
-        </joint>
+        </xacro:axis_dome_ptz>
       </xacro:if>
       <!-- Rear Axis PTZ camera -->
       <xacro:if value="$(arg rear_axis_ptz_enable)">
-        <link name="rear_axis_ptz_camera_link"/>
-        <joint name="rear_axis_to_base" type="fixed">
-          <parent link="base_link" />
-          <child link="rear_axis_ptz_camera_link" />
+        <xacro:axis_dome_ptz prefix="axis_rear_ptz_camera" parent="base_link" topic="/sensors/camera_$(arg rear_axis_ptz_num)/image_raw">
           <origin xyz="$(arg rear_axis_ptz_xyz)" rpy="$(arg rear_axis_ptz_rpy)"/>
-        </joint>
+        </xacro:axis_dome_ptz>
       </xacro:if>
       <!-- Axis Q62 PTZ camera -->
       <xacro:if value="$(arg axis_q62_enable)">
-        <xacro:axis_q62 prefix="ptz_camera" parent="base_link" axis_ptz_num="$(arg axis_ptz_num)">
+        <xacro:axis_q62 prefix="ptz_camera" parent="base_link" topic="/sensors/camera_$(arg axis_ptz_num)/image_raw">
           <origin xyz="$(arg axis_q62_xyz)" rpy="$(arg axis_q62_rpy)" />
         </xacro:axis_q62>

Commit message: added antenna links to urdf

File: urdf/outdoornav_description.urdf.xacro (robot description, xacro)
@@ -69,4 +69,8 @@
     <xacro:arg name="xvn_xyz"                  default="$(optenv XVN_XYZ 0 0 0)" />
     <xacro:arg name="xvn_rpy"                  default="$(optenv XVN_RPY 0 0 0)" />
+    <xacro:arg name="xvn_gnss1_xyz"            default="$(optenv XVN_GNSS1_XYZ 0 0 0)" />
+    <xacro:arg name="xvn_gnss1_rpy"            default="$(optenv XVN_GNSS1_RPY 0 0 0)" />
+    <xacro:arg name="xvn_gnss2_xyz"            default="$(optenv XVN_GNSS2_XYZ 0 0 0)" />
+    <xacro:arg name="xvn_gnss2_rpy"            default="$(optenv XVN_GNSS2_RPY 0 0 0)" />
     <xacro:arg name="onav_urdf_extras"         default="$(optenv OUTDOORNAV_URDF_EXTRAS empty.urdf)" />
     <xacro:arg name="enable_docking"           default="$(optenv OUTDOORNAV_ENABLE_DOCKING false)" />
@@ -239,4 +243,16 @@
           <origin xyz="$(arg xvn_xyz)" rpy="$(arg xvn_rpy)"/>
         </joint>
+        <link name="gps_position_link"/>
+        <joint name="xvn_gnss1_base" type="fixed">
+          <parent link="base_link" />
+          <child link="gps_position_link" />
+          <origin xyz="$(arg xvn_gnss1_xyz)" rpy="$(arg xvn_gnss1_rpy)"/>
+        </joint>
+        <link name="gps_heading_link"/>
+        <joint name="xvn_gnss2_base" type="fixed">
+          <parent link="base_link" />
+          <child link="gps_heading_link" />
+          <origin xyz="$(arg xvn_gnss2_xyz)" rpy="$(arg xvn_gnss2_rpy)"/>
+        </joint>
       </xacro:if>
       <!-- Microstrain Link -->

Commit message: added hesai lidar link to urdf

File: urdf/outdoornav_description.urdf.xacro (robot description, xacro)
@@ -53,4 +53,8 @@
     <xacro:arg name="rear_vlp_xyz"             default="$(optenv REAR_VLP_XYZ 0.0 0.0 0.0)" />
     <xacro:arg name="rear_vlp_rpy"             default="$(optenv REAR_VLP_RPY 0.0 0.0 0.0)" />
+    <xacro:arg name="hesai_enable"             default="$(optenv HESAI_ENABLE_DRIVER false)" />
+    <xacro:arg name="hesai_xyz"                default="$(optenv HESAI_XYZ 0.0 0.0 0.0)" />
+    <xacro:arg name="hesai_rpy"                default="$(optenv HESAI_RPY 0.0 0.0 0.0)" />
+    <xacro:arg name="hesai_num"                default="$(optenv HESAI_NUM 0)" />
     <xacro:arg name="d435_enable"              default="$(optenv D435_ENABLE_DRIVER false)" />
     <xacro:arg name="d435_xyz"                 default="$(optenv D435_XYZ 0.0 0.0 0.0)" />
@@ -295,4 +299,13 @@
         </xacro:VLP-16>
       </xacro:if>
+      <!-- Hesai Link -->
+      <xacro:if value="$(arg hesai_enable)">
+        <link name="hesai_lidar"/>
+        <joint name="hesai_to_base" type="fixed">
+          <parent link="base_link" />
+          <child link="hesai_lidar" />
+          <origin xyz="$(arg hesai_xyz)" rpy="$(arg hesai_rpy)"/>
+        </joint>
+      </xacro:if>
       <!-- 2D LiDAR(s) Link -->
       <xacro:if value="$(arg lms1xx_enable)">

Commit message: added microstrain gnss links

File: urdf/outdoornav_description.urdf.xacro (robot description, xacro)
@@ -16,6 +16,11 @@
     <xacro:arg name="ublox_rpy"                default="$(optenv UBLOX_POSITION_GPS_RPY 0.0 0.0 0.0)" />
     <xacro:arg name="microstrain_enable"       default="$(optenv MICROSTRAIN_ENABLE_DRIVER false)" />
+    <xacro:arg name="microstrain_gnss_enable"  default="$(optenv MICROSTRAIN_ENABLE_GNSS false )" />
     <xacro:arg name="microstrain_xyz"          default="$(optenv MICROSTRAIN_XYZ 0.0 0.0 0.0)" />
     <xacro:arg name="microstrain_rpy"          default="$(optenv MICROSTRAIN_RPY 0.0 0.0 0.0)" />
+    <xacro:arg name="microstrain_gnss1_xyz"    default="$(optenv MICROSTRAIN_GNSS1_XYZ 0.0 0.0 0.0)" />
+    <xacro:arg name="microstrain_gnss1_rpy"    default="$(optenv MICROSTRAIN_GNSS1_RPY 0.0 0.0 0.0)" />
+    <xacro:arg name="microstrain_gnss2_xyz"    default="$(optenv MICROSTRAIN_GNSS2_XYZ 0.0 0.0 0.0)" />
+    <xacro:arg name="microstrain_gnss2_rpy"    default="$(optenv MICROSTRAIN_GNSS2_RPY 0.0 0.0 0.0)" />
     <xacro:arg name="xsens_enable"             default="$(optenv XSENS_ENABLE_DRIVER false)" />
     <xacro:arg name="xsens_xyz"                default="$(optenv XSENS_XYZ 0.0 0.0 0.0)" />
@@ -277,4 +282,18 @@
           <origin xyz="$(arg microstrain_xyz)" rpy="$(arg microstrain_rpy)"/>
         </joint>
+        <xacro:if value="${arg microstrain_gnss_enable">
+          <link name="gps_position_link"/>
+          <joint name="gnss1_to_microstrain" type="fixed">
+            <parent link="microstrain_link" />
+            <child link="gps_position_link" />
+            <origin xyz="$(arg microstrain_gnss1_xyz)" rpy="$(arg microstrain_gnss1_rpy)"/>
+          </joint>
+          <link name="gps_heading_link"/>
+          <joint name="gnss2_to_microstrain" type="fixed">
+            <parent link="microstrain_link" />
+            <child link="gps_heading_link" />
+            <origin xyz="$(arg microstrain_gnss2_xyz)" rpy="$(arg microstrain_gnss2_rpy)"/>
+          </joint>
+        </xacro:if>
       </xacro:if>
       <!-- Xsens Link -->

Commit message: added ouster lidar link/joint to urdf

File: urdf/outdoornav_description.urdf.xacro (robot description, xacro)
@@ -62,4 +62,7 @@
     <xacro:arg name="hesai_rpy"                default="$(optenv HESAI_RPY 0.0 0.0 0.0)" />
     <xacro:arg name="hesai_num"                default="$(optenv HESAI_NUM 0)" />
+    <xacro:arg name="ouster_enable"            default="$(optenv OUSTER_ENABLE_DRIVER false)" />
+    <xacro:arg name="ouster_xyz"               default="$(optenv OUSTER_XYZ 0.0 0.0 0.0)" />
+    <xacro:arg name="ouster_rpy"               default="$(optenv OUSTER_RPY 0.0 0.0 0.0)" />
     <xacro:arg name="d435_enable"              default="$(optenv D435_ENABLE_DRIVER false)" />
     <xacro:arg name="d435_xyz"                 default="$(optenv D435_XYZ 0.0 0.0 0.0)" />
@@ -327,5 +330,14 @@
         </joint>
       </xacro:if>
-      <!-- 2D LiDAR(s) Link -->
+      <!-- Ouster Link -->
+      <xacro:if value="$(arg ouster_enable)">
+        <link name="ouster_lidar"/>
+        <joint name="ouster_to_base" type="fixed">
+          <parent link="base_link" />
+          <child link="ouster_lidar" />
+          <origin xyz="$(arg ouster_xyz)" rpy="$(arg ouster_rpy)"/>
+        </joint>
+      </xacro:if>
+      <!-- 2D LiDAR Link(s) -->
       <xacro:if value="$(arg lms1xx_enable)">
         <xacro:sick_lms1xx_mount prefix="front" parent="base_link" topic="/sensors/lidar_$(arg lms1xx_num)/scan" tower="0" robot_namespace="/">

Commit message: use updated ouster driver and description repos

File: urdf/outdoornav_description.urdf.xacro (robot description, xacro)
@@ -54,5 +54,5 @@
     <xacro:arg name="vlp_xyz"                  default="$(optenv VLP_XYZ 0.0 0.0 0.0)" />
     <xacro:arg name="vlp_rpy"                  default="$(optenv VLP_RPY 0.0 0.0 0.0)" />
-    <xacro:arg name="vlp_num"                  default="$(optenv VLP_NUM 0)" />
+    <xacro:arg name="vlp_num"                  default="$(optenv VLP_LIDAR_NUM 0)" />
     <xacro:arg name="rear_vlp_enable"          default="$(optenv REAR_VLP_ENABLE_DRIVER false)" />
     <xacro:arg name="rear_vlp_xyz"             default="$(optenv REAR_VLP_XYZ 0.0 0.0 0.0)" />
@@ -65,4 +65,6 @@
     <xacro:arg name="ouster_xyz"               default="$(optenv OUSTER_XYZ 0.0 0.0 0.0)" />
     <xacro:arg name="ouster_rpy"               default="$(optenv OUSTER_RPY 0.0 0.0 0.0)" />
+    <xacro:arg name="ouster_lidar_num"         default="$(optenv OUSTER_LIDAR_NUM 0)" />
+    <xacro:arg name="ouster_imu_num"           default="$(optenv OUSTER_IMU_NUM 0)" />
     <xacro:arg name="d435_enable"              default="$(optenv D435_ENABLE_DRIVER false)" />
     <xacro:arg name="d435_xyz"                 default="$(optenv D435_XYZ 0.0 0.0 0.0)" />
@@ -332,10 +334,7 @@
       <!-- Ouster Link -->
       <xacro:if value="$(arg ouster_enable)">
-        <link name="ouster_lidar"/>
-        <joint name="ouster_to_base" type="fixed">
-          <parent link="base_link" />
-          <child link="ouster_lidar" />
-          <origin xyz="$(arg ouster_xyz)" rpy="$(arg ouster_rpy)"/>
-        </joint>
+        <xacro:VLP-16 name="os_sensor" parent="base_link" topic_points="/sensors/lidar_$(arg ouster_lidar_num)/pointcloud" topic_imu="/sensors/imu_$(arg ouster_imu_num)/data">
+          <origin xyz="$(arg ouster_xyz)" rpy="$(arg ouster_rpy)" />
+        </xacro:VLP-16>
       </xacro:if>
       <!-- 2D LiDAR Link(s) -->
