Commit message: remove circular dependency by adding local copies of accesory urdf files

File: urdf/accessories/sick_lms1xx_mount.urdf.xacro (robot description, xacro)
@@ -38,5 +38,5 @@
           <geometry>
             <!-- Origin of this mesh is the base of the bracket. -->
-            <mesh filename="package://husky_description/meshes/accessories/lms1xx_mount.dae" />
+            <mesh filename="package://cpr_onav_description/meshes/accessories/lms1xx_mount.dae" />
           </geometry>
         </visual>

File: urdf/outdoornav_description.urdf.xacro (robot description, xacro)
@@ -94,6 +94,6 @@
     <xacro:if value="${outdoornav_configuration == 'custom'}">
       <xacro:include filename="$(find velodyne_description)/urdf/VLP-16.urdf.xacro"/>
-      <xacro:include filename="$(find husky_description)/urdf/accessories/hokuyo_ust10.urdf.xacro" />
-      <xacro:include filename="$(find husky_description)/urdf/accessories/sick_lms1xx_mount.urdf.xacro"/>
+      <xacro:include filename="$(find cpr_onav_description)/urdf/accessories/hokuyo_ust10.urdf.xacro" />
+      <xacro:include filename="$(find cpr_onav_description)/urdf/accessories/sick_lms1xx_mount.urdf.xacro"/>
       <xacro:include filename="$(find realsense2_description)/urdf/_d435.urdf.xacro" />
       <!-- Position GPS (Duro) -->
