Commit message: Fix the path for the Hokuyo mesh, add simplified collision geometry

File: urdf/accessories/hokuyo_ust10.urdf.xacro (robot description, xacro)
@@ -58,8 +58,20 @@
         <geometry>
           <!-- Origin of this mesh is the base of the bracket. -->
-          <mesh filename="package://cpr_onav_description/meshes/accessories/hokuyo_ust10.stl" />
+          <mesh filename="package://cpr_onav_description/meshes/hokuyo_ust10.stl" />
         </geometry>
         <material name="dark_grey" />
       </visual>
+      <collision>
+        <origin xyz="0 0 0.0175" rpy="0 0 0" />
+        <geometry>
+          <box size="0.05 0.05 0.035" />
+        </geometry>
+      </collision>
+      <collision>
+        <origin xyz="0 0 0.035" rpy="0 0 0" />
+        <geometry>
+          <cylinder radius="0.024" length="0.07" />
+        </geometry>
+      </collision>
     </link>
     <joint name="${prefix}_laser_joint" type="fixed">

Commit message: Mod: Decrease Hokuyo update rate from 50->10 Hz
Signed-off-by: Stephen Phillips <stphillips@clearpathrobotics.com>

File: urdf/accessories/hokuyo_ust10.urdf.xacro (robot description, xacro)
@@ -2,5 +2,5 @@
 <robot xmlns:xacro="http://ros.org/wiki/xacro">
   <xacro:macro name="hokuyo_ust10_mount" params="prefix topic parent_link min_angle:=-2.35619 max_angle:=2.35619 *origin">
-    <xacro:macro name="hokuyo_ust10" params="frame:=laser topic:=scan sample_size:=720 update_rate:=50
+    <xacro:macro name="hokuyo_ust10" params="frame:=laser topic:=scan sample_size:=720 update_rate:=10
                min_angle:=${min_angle} max_angle:=${max_angle} min_range:=0.1 max_range:=30.0 robot_namespace:=/">
       <link name="${frame}">
