Commit message: Invert the direction of the pan so that positive is clockwise

File: urdf/accessories/axis_q62.urdf.xacro (robot description, xacro)
@@ -43,5 +43,5 @@
     </link>
     <joint name="${prefix}_pan_joint" type="continuous">
-      <axis xyz="0 0 1" />
+      <axis xyz="0 0 -1" />
       <parent link="${prefix}_base_link" />
       <child link="${prefix}_body_link" />
